File: guhPLC_V0.1.sch (EAGLE design)
At the start: 170 parts, among them IC1 7812DT, K1 62104021021, K2 62104021021, K4 62101021021, K5 61900611021, Q1 BSS123, Q10 BSS123, Q11 BSS123, Q3 32.768k, Q4 BSS123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

Commit message: added pull ups for i2C changed the port for the 32kHz crystal at STM32
Parts:
- added R25, R26: 10k, resistor:R-EU_R0603
Connections:
- net +3V3: now also R25.2, R26.2
- net OSCI: now also U$2.PC14/OSC32_IN; no longer U$2.PF0/OSC_IN
- net OSCO: now also U$2.PC15/OSC32_OUT; no longer U$2.PF1/OSC_OUT
- net SCL: now also R25.1
- net SDA: now also R26.1
Changed lines of the file:
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@@
 <part name="GND2" library="supply1" deviceset="GND" device=""/>
 <part name="GND26" library="supply1" deviceset="GND" device=""/>
+<part name="+3V9" library="supply1" deviceset="+3V3" device=""/>
+<part name="+3V21" library="supply1" deviceset="+3V3" device=""/>
+<part name="R25" library="resistor" deviceset="R-EU_" device="R0603" value="10k"/>
+<part name="R26" library="resistor" deviceset="R-EU_" device="R0603" value="10k"/>
 </parts>
 <sheets>
@@
 <instance part="GND2" gate="1" x="91.44" y="246.38" rot="R90"/>
 <instance part="GND26" gate="1" x="200.66" y="246.38" rot="R90"/>
+<instance part="+3V9" gate="G$1" x="492.76" y="182.88"/>
+<instance part="+3V21" gate="G$1" x="500.38" y="182.88"/>
+<instance part="R25" gate="G$1" x="492.76" y="172.72" rot="R90"/>
+<instance part="R26" gate="G$1" x="500.38" y="172.72" rot="R90"/>
 </instances>
 <busses>
@@
 <segment>
 <pinref part="U$2" gate="G$1" pin="PB9/I2C1_SDA/TIM17_CH1/CAN_TX"/>
-<wire x1="467.36" y1="162.56" x2="485.14" y2="162.56" width="0.1524" layer="91"/>
-<label x="472.44" y="162.56" size="1.778" layer="95"/>
+<wire x1="467.36" y1="162.56" x2="500.38" y2="162.56" width="0.1524" layer="91"/>
+<label x="502.92" y="162.56" size="1.778" layer="95"/>
+<pinref part="R26" gate="G$1" pin="1"/>
+<wire x1="500.38" y1="162.56" x2="510.54" y2="162.56" width="0.1524" layer="91"/>
+<wire x1="500.38" y1="167.64" x2="500.38" y2="162.56" width="0.1524" layer="91"/>
+<junction x="500.38" y="162.56"/>
 </segment>
 <segment>
@@
 <segment>
 <pinref part="U$2" gate="G$1" pin="PB8/I2C1_SCL/TIM16_CH1/CAN_RX"/>
-<wire x1="467.36" y1="165.1" x2="485.14" y2="165.1" width="0.1524" layer="91"/>
-<label x="472.44" y="165.1" size="1.778" layer="95"/>
+<wire x1="467.36" y1="165.1" x2="492.76" y2="165.1" width="0.1524" layer="91"/>
+<label x="502.92" y="165.1" size="1.778" layer="95"/>
+<pinref part="R25" gate="G$1" pin="1"/>
+<wire x1="492.76" y1="165.1" x2="510.54" y2="165.1" width="0.1524" layer="91"/>
+<wire x1="492.76" y1="167.64" x2="492.76" y2="165.1" width="0.1524" layer="91"/>
+<junction x="492.76" y="165.1"/>
 </segment>
 <segment>
@@
 <net name="OSCI" class="0">
 <segment>
-<pinref part="U$2" gate="G$1" pin="PF0/OSC_IN"/>
-<wire x1="373.38" y1="165.1" x2="360.68" y2="165.1" width="0.1524" layer="91"/>
-<label x="363.22" y="165.1" size="1.778" layer="95"/>
-</segment>
-<segment>
 <pinref part="Q3" gate="G$1" pin="2"/>
 <wire x1="269.24" y1="226.06" x2="284.48" y2="226.06" width="0.1524" layer="91"/>
@@
 <label x="269.24" y="226.06" size="1.778" layer="95"/>
 </segment>
+<segment>
+<pinref part="U$2" gate="G$1" pin="PC14/OSC32_IN"/>
+<wire x1="373.38" y1="149.86" x2="360.68" y2="149.86" width="0.1524" layer="91"/>
+<label x="363.22" y="149.86" size="1.778" layer="95"/>
+</segment>
 </net>
 <net name="ADC2" class="0">
@@
 <wire x1="-22.86" y1="20.32" x2="2.54" y2="20.32" width="0.1524" layer="91"/>
 </segment>
+<segment>
+<pinref part="+3V9" gate="G$1" pin="+3V3"/>
+<pinref part="R25" gate="G$1" pin="2"/>
+<wire x1="492.76" y1="180.34" x2="492.76" y2="177.8" width="0.1524" layer="91"/>
+</segment>
+<segment>
+<pinref part="+3V21" gate="G$1" pin="+3V3"/>
+<pinref part="R26" gate="G$1" pin="2"/>
+<wire x1="500.38" y1="180.34" x2="500.38" y2="177.8" width="0.1524" layer="91"/>
+</segment>
 </net>
 <net name="UC_INT" class="0">
@@
 <net name="OSCO" class="0">
 <segment>
-<pinref part="U$2" gate="G$1" pin="PF1/OSC_OUT"/>
-<wire x1="373.38" y1="162.56" x2="360.68" y2="162.56" width="0.1524" layer="91"/>
-<label x="363.22" y="162.56" size="1.778" layer="95"/>
-</segment>
-<segment>
 <pinref part="Q3" gate="G$1" pin="1"/>
 <wire x1="284.48" y1="218.44" x2="284.48" y2="215.9" width="0.1524" layer="91"/>
@@
 <junction x="284.48" y="215.9"/>
 </segment>
+<segment>
+<pinref part="U$2" gate="G$1" pin="PC15/OSC32_OUT"/>
+<wire x1="373.38" y1="147.32" x2="360.68" y2="147.32" width="0.1524" layer="91"/>
+<label x="363.22" y="147.32" size="1.778" layer="95"/>
+</segment>
 </net>

Commit message: Added License to README Minor bug fixes
Parts:
- C16, C17: device resistor:C-EUC0805 -> resistor:C-EUC0603
- C25, C26, C31: device resistor:C-EUC0402 -> resistor:C-EUC0603
- C3: device resistor:C-EUC1206 -> resistor:C-EUC0603
- C4, C5: value 10n -> 10p; device resistor:C-EUC0402K -> resistor:C-EUC0603
- C6: device resistor:C-EUC1206 -> resistor:C-EUC0504
- D1, D11, D13, D15, D17, D19, D20, D21, D22, D23, D24, D25, D26, D4, D7, D9: value CGRM4001-G -> 1N4148W-7-F; device diode:CGRM4001-G -> guh:1N4148W-7-F
Other:
- moved on the sheet: D24, IC1

Commit message: Added 1-wire interface
Parts:
- added C33: 100n, resistor:C-EUC0603
- added IC2: DS2482S-100SOI, guh:DS2482S-100SOI
- added Q12: FDN360P, transistor-power:FDN360P
- added R31: 10, resistor:R-EU_R0805
Connections:
- new net 1-WIRE: IC2.IO, Q12.D, X2-6.KL
- new net N$19: Q12.S, R31.1
- new net N$2: IC2.PCTLZ, Q12.G
- net +3V3: now also C33.2, IC2.VCC, R31.2
- net GND: now also C33.1, IC2.AD0, IC2.AD1, IC2.GND; no longer X2-6.KL
- net SCL: now also IC2.SCL
- net SDA: now also IC2.SDA
Other:
- note added: "1-Wire"
Changed lines of the file:
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@@
 <part name="D17" library="guh" deviceset="1N4148W-7-F" device=""/>
 <part name="D19" library="guh" deviceset="1N4148W-7-F" device=""/>
+<part name="IC2" library="guh" deviceset="DS2482S-100" device="SOI"/>
+<part name="+3V22" library="supply1" deviceset="+3V3" device=""/>
+<part name="GND27" library="supply1" deviceset="GND" device=""/>
+<part name="GND28" library="supply1" deviceset="GND" device=""/>
+<part name="C33" library="resistor" deviceset="C-EU" device="C0603" value="100n"/>
+<part name="GND29" library="supply1" deviceset="GND" device=""/>
+<part name="R31" library="resistor" deviceset="R-EU_" device="R0805" value="10"/>
+<part name="+3V23" library="supply1" deviceset="+3V3" device=""/>
+<part name="Q12" library="transistor-power" deviceset="FDN360P" device=""/>
 </parts>
 <sheets>
@@
 <text x="360.68" y="480.06" size="6.4516" layer="94">Licensed under CERN v1.2</text>
 <text x="360.68" y="467.36" size="6.4516" layer="94">ARGE guh</text>
+<text x="-93.98" y="142.24" size="6.4516" layer="97">1-Wire</text>
+<wire x1="71.12" y1="152.4" x2="248.92" y2="152.4" width="0.1524" layer="97"/>
 </plain>
 <instances>
@@
 <instance part="X6" gate="-9" x="449.58" y="274.32"/>
 <instance part="X6" gate="-10" x="449.58" y="269.24"/>
-<instance part="GND70" gate="1" x="124.46" y="302.26" rot="R270"/>
+<instance part="GND70" gate="1" x="124.46" y="299.72" rot="R270"/>
 <instance part="GND71" gate="1" x="137.16" y="284.48" rot="R270"/>
 <instance part="GND72" gate="1" x="137.16" y="269.24" rot="R270"/>
@@
 <instance part="D17" gate="G$1" x="195.58" y="60.96" rot="R90"/>
 <instance part="D19" gate="G$1" x="195.58" y="25.4" rot="R90"/>
+<instance part="IC2" gate="G$1" x="-22.86" y="127"/>
+<instance part="+3V22" gate="G$1" x="-43.18" y="144.78"/>
+<instance part="GND27" gate="1" x="-43.18" y="124.46" rot="R270"/>
+<instance part="GND28" gate="1" x="2.54" y="132.08" rot="R90"/>
+<instance part="C33" gate="G$1" x="-53.34" y="134.62" rot="R90"/>
+<instance part="GND29" gate="1" x="-60.96" y="134.62" rot="R270"/>
+<instance part="R31" gate="G$1" x="25.4" y="134.62" rot="R90"/>
+<instance part="+3V23" gate="G$1" x="25.4" y="144.78"/>
+<instance part="Q12" gate="G$1" x="22.86" y="121.92"/>
 </instances>
 <busses>
@@
 <pinref part="X2" gate="-3" pin="KL"/>
 <wire x1="157.48" y1="304.8" x2="139.7" y2="304.8" width="0.1524" layer="91"/>
-<wire x1="139.7" y1="304.8" x2="139.7" y2="302.26" width="0.1524" layer="91"/>
+<wire x1="139.7" y1="304.8" x2="139.7" y2="299.72" width="0.1524" layer="91"/>
 <pinref part="X2" gate="-4" pin="KL"/>
-<wire x1="139.7" y1="302.26" x2="139.7" y2="299.72" width="0.1524" layer="91"/>
 <wire x1="139.7" y1="299.72" x2="157.48" y2="299.72" width="0.1524" layer="91"/>
 <pinref part="GND70" gate="1" pin="GND"/>
-<wire x1="127" y1="302.26" x2="139.7" y2="302.26" width="0.1524" layer="91"/>
-<junction x="139.7" y="302.26"/>
+<wire x1="127" y1="299.72" x2="139.7" y2="299.72" width="0.1524" layer="91"/>
+<junction x="139.7" y="299.72"/>
+<pinref part="X2" gate="-5" pin="KL"/>
+<wire x1="157.48" y1="294.64" x2="139.7" y2="294.64" width="0.1524" layer="91"/>
+<wire x1="139.7" y1="294.64" x2="139.7" y2="299.72" width="0.1524" layer="91"/>
+<junction x="139.7" y="299.72"/>
 </segment>
 <segment>
@@
 <wire x1="157.48" y1="284.48" x2="139.7" y2="284.48" width="0.1524" layer="91"/>
 <pinref part="GND71" gate="1" pin="GND"/>
-<pinref part="X2" gate="-5" pin="KL"/>
-<wire x1="157.48" y1="294.64" x2="139.7" y2="294.64" width="0.1524" layer="91"/>
-<wire x1="139.7" y1="294.64" x2="139.7" y2="289.56" width="0.1524" layer="91"/>
-<pinref part="X2" gate="-6" pin="KL"/>
-<wire x1="139.7" y1="289.56" x2="157.48" y2="289.56" width="0.1524" layer="91"/>
-<wire x1="139.7" y1="284.48" x2="139.7" y2="289.56" width="0.1524" layer="91"/>
-<junction x="139.7" y="284.48"/>
-<junction x="139.7" y="289.56"/>
 </segment>
 <segment>
@@
 <pinref part="GND2" gate="1" pin="GND"/>
 </segment>
+<segment>
+<pinref part="IC2" gate="G$1" pin="GND"/>
+<pinref part="GND27" gate="1" pin="GND"/>
+<wire x1="-35.56" y1="124.46" x2="-40.64" y2="124.46" width="0.1524" layer="91"/>
+</segment>
+<segment>
+<pinref part="GND28" gate="1" pin="GND"/>
+<wire x1="0" y1="132.08" x2="-2.54" y2="132.08" width="0.1524" layer="91"/>
+<wire x1="-2.54" y1="132.08" x2="-2.54" y2="134.62" width="0.1524" layer="91"/>
+<pinref part="IC2" gate="G$1" pin="AD0"/>
+<wire x1="-2.54" y1="134.62" x2="-10.16" y2="134.62" width="0.1524" layer="91"/>
+<pinref part="IC2" gate="G$1" pin="AD1"/>
+<wire x1="-10.16" y1="129.54" x2="-2.54" y2="129.54" width="0.1524" layer="91"/>
+<wire x1="-2.54" y1="129.54" x2="-2.54" y2="132.08" width="0.1524" layer="91"/>
+<junction x="-2.54" y="132.08"/>
+</segment>
+<segment>
+<pinref part="C33" gate="G$1" pin="1"/>
+<pinref part="GND29" gate="1" pin="GND"/>
+<wire x1="-55.88" y1="134.62" x2="-58.42" y2="134.62" width="0.1524" layer="91"/>
+</segment>
 </net>
 <net name="VCC" class="1">
@@
 <label x="220.98" y="474.98" size="1.9304" layer="95"/>
 </segment>
+<segment>
+<pinref part="IC2" gate="G$1" pin="SDA"/>
+<wire x1="-10.16" y1="119.38" x2="10.16" y2="119.38" width="0.1524" layer="91"/>
+<label x="0" y="119.38" size="1.778" layer="95"/>
+</segment>
 </net>
 <net name="SCL" class="0">
@@
 <label x="220.98" y="477.52" size="1.9304" layer="95"/>
 </segment>
+<segment>
+<pinref part="IC2" gate="G$1" pin="SCL"/>
+<wire x1="-35.56" y1="119.38" x2="-58.42" y2="119.38" width="0.1524" layer="91"/>
+<label x="-55.88" y="119.38" size="1.778" layer="95"/>
+</segment>
 </net>
 <net name="OSCI" class="0">
@@
 <wire x1="500.38" y1="180.34" x2="500.38" y2="177.8" width="0.1524" layer="91"/>
 </segment>
+<segment>
+<pinref part="IC2" gate="G$1" pin="VCC"/>
+<pinref part="+3V22" gate="G$1" pin="+3V3"/>
+<wire x1="-35.56" y1="134.62" x2="-43.18" y2="134.62" width="0.1524" layer="91"/>
+<wire x1="-43.18" y1="134.62" x2="-43.18" y2="142.24" width="0.1524" layer="91"/>
+<pinref part="C33" gate="G$1" pin="2"/>
+<wire x1="-43.18" y1="134.62" x2="-48.26" y2="134.62" width="0.1524" layer="91"/>
+<junction x="-43.18" y="134.62"/>
+</segment>
+<segment>
+<pinref part="+3V23" gate="G$1" pin="+3V3"/>
+<pinref part="R31" gate="G$1" pin="2"/>
+<wire x1="25.4" y1="142.24" x2="25.4" y2="139.7" width="0.1524" layer="91"/>
+</segment>
 </net>
 <net name="UC_INT" class="0">
@@
 <wire x1="373.38" y1="175.26" x2="355.6" y2="175.26" width="0.1524" layer="91"/>
 <pinref part="R24" gate="G$1" pin="2"/>
-<wire x1="355.6" y1="175.26" x2="342.9" y2="175.26" width="0.1524" layer="91"/>
-<junction x="355.6" y="175.26"/>
-<label x="342.9" y="175.26" size="1.778" layer="95"/>
+<label x="358.14" y="175.26" size="1.778" layer="95"/>
 </segment>
 </net>
@@
 </segment>
 </net>
+<net name="1-WIRE" class="0">
+<segment>
+<pinref part="IC2" gate="G$1" pin="IO"/>
+<wire x1="-35.56" y1="129.54" x2="-58.42" y2="129.54" width="0.1524" layer="91"/>
+<label x="-55.88" y="129.54" size="1.778" layer="95"/>
+</segment>
+<segment>
+<pinref part="X2" gate="-6" pin="KL"/>
+<wire x1="139.7" y1="289.56" x2="157.48" y2="289.56" width="0.1524" layer="91"/>
+<label x="142.24" y="289.56" size="1.778" layer="95"/>
+</segment>
+<segment>
+<wire x1="25.4" y1="114.3" x2="45.72" y2="114.3" width="0.1524" layer="91"/>
+<label x="35.56" y="114.3" size="1.778" layer="95"/>
+<pinref part="Q12" gate="G$1" pin="D"/>
+<wire x1="25.4" y1="116.84" x2="25.4" y2="114.3" width="0.1524" layer="91"/>
+</segment>
+</net>
+<net name="N$2" class="0">
+<segment>
+<pinref part="IC2" gate="G$1" pin="PCTLZ"/>
+<pinref part="Q12" gate="G$1" pin="G"/>
+<wire x1="-10.16" y1="124.46" x2="20.32" y2="124.46" width="0.1524" layer="91"/>
+</segment>
+</net>
+<net name="N$19" class="0">
+<segment>
+<pinref part="R31" gate="G$1" pin="1"/>
+<pinref part="Q12" gate="G$1" pin="S"/>
+<wire x1="25.4" y1="129.54" x2="25.4" y2="127" width="0.1524" layer="91"/>
+</segment>
+</net>
