File: guhPLC_V0.2.brd (EAGLE design)
At the start: 156 x 86.5 mm, 176 parts, among them IC1 7812DT, IC2 DS2482S-100SOI, K1 62104021021, K2 62104021021, K4 62101021021, K5 61900611021, Q1 BSS123, Q10 BSS123, Q11 BSS123, Q12 FDN360P, Q3 32.768k, Q4 BSS123, Q5 BSS123, Q6 BSS123, Q7 BSS123, Q8 BSS123, Q9 BSS123, U1 LM2672M-3.3, U3 TLC272CD, U4 TLC272CD, U5 ENC28J60/SS, U6 SN65HVD75D, X1 J1006F01P, X2 MKDSN1,5/10-5,08, X3 MKDSN1,5/10-5,08, X4 MKDSN1,5/10-5,08, X5 MKDSN1,5/10-5,08, X6 MKDSN1,5/10-5,08

Commit message: Changed RS485 to CAN Bus - for better multi master communication
Parts:
- removed Q11: BSS123, transistor-small-signal:SOT23
- removed R68, R69: 10, resistor:R0603
- removed R70, R71, R72: 10k, resistor:R0603
- removed U6: SN65HVD75D, guh:SOIC127P600X175-8N
- added C34: 100n, resistor:C0603
- added C35, C36: 9pF, resistor:C0603
- added C37, C38: 10u, resistor:C1206
- added Q2: E3SB16.0000F09G11AE, guh:E3SBXXXXXXXF09G11AE
- added R34, R36, R38: 10k, resistor:R0603
- added R37: 18k, resistor:R0603
- added U$3: MCP2515-I/SO, guh:SOIC127P1034X264-18N
- added U$4: MCP2551-I/SN, guh:SOIC127P600X175-8N
- added U2: LD6815TD/18P, guh:SOT95P275X110-5N
- C6: device resistor:C0504 -> resistor:C0603
- moved C6 16.2 mm to (2.00, 37.0)
- moved D5 11.6 mm to (30.1, 13.9), turned to 90 degrees
- moved R31 8.85 mm to (15.0, 44.5), turned to 180 degrees
- moved F1 8.25 mm to (16.2, 11.0)
- moved C33 6.95 mm to (18.5, 51.5)
- moved IC2 6.95 mm to (12.5, 53.5)
- moved Q12 6.95 mm to (15.0, 48.0)
- moved C14 3.74 mm to (55.3, 19.8), turned to 180 degrees
- moved C15 2.24 mm to (40.8, 20.0)
- moved D2 1.58 mm to (54.8, 26.2)
- moved U1 1.50 mm to (47.3, 24.8)
- moved C3 1.00 mm to (47.4, 28.5)
- moved C5 1.00 mm to (104.7, 49.8)
- moved L1 0.50 mm to (47.3, 34.7)
- moved R24 0.50 mm to (116.0, 59.0), turned to 270 degrees
Connections:
- removed net CS: K4.1, U5.9
- removed net DIR: Q11.3, R72.2, U6.2, U6.3
- removed net MISO: K4.4, U5.6
- removed net MOSI: K4.3, U5.7
- removed net N$63: R68.1, U6.7
- removed net N$64: R69.1, U6.6
- removed net N$65: Q11.1, R70.1
- removed net RS485_A: R69.2, X2.8
- removed net RS485_B: R68.2, X2.9
- removed net RX: K1.35, R71.1, U6.1
- removed net SCK: K4.2, U5.8
- removed net TX: K1.34, R70.2, U6.4
- new net +5V: C38.1, C6.1, U$4.3, U2.5
- new net CANH: U$4.7, X2.7
- new net CANL: U$4.6, X2.6
- new net CAN_INT: U$3.12
- new net CAN_NRST: R34.2, U$3.17
- new net CAN_OSC1: C35.1, Q2.1, U$3.8
- new net CAN_OSC2: C36.1, Q2.3, U$3.7
- new net CAN_RX: R36.2, U$4.4
- new net N$20: U$3.1, U$4.1
- new net N$22: R36.1, R37.1, U$3.2
- new net N$24: R38.2, U$4.8
- new net SOM_NRST: K1.2, U$2.28
- new net SPI2_CLK: K4.2, U$3.13
- new net SPI2_CS0: K4.1, U$3.16
- new net SPI2_MISO: K4.4, U$3.15
- new net SPI2_MOSI: K4.3, U$3.14
- new net SPI_CLK: K1.13, U5.8
- new net SPI_CS0: K1.14, U5.9
- new net SPI_MISO: K1.12, U5.6
- new net SPI_MOSI: K1.11, U5.7
- net +3V3: now also C34.1, R34.1, U$3.18; no longer C6.1, R71.2, R72.1, U6.8
- net 1-WIRE: now also X2.9; no longer X2.6
- net GND: now also C34.2, C35.2, C36.2, C37.2, C38.2, Q2.2, Q2.4, R37.2, R38.1, U$3.9, U$4.2, U2.2, X2.8; no longer Q11.2, U6.5, X2.7
- net VCC: now also C37.1, U2.1, U2.3
Routing:
- net SOM_NRST: track 0.00 -> 136.1 mm, vias 0 -> 2
- net TX: track 76.2 -> 0.00 mm
- net UC_BOOT: track 76.7 -> 5.75 mm, vias 1 -> 0
- net RX: track 68.7 -> 0.00 mm, vias 2 -> 0
- net +5V: track 0.00 -> 44.5 mm, vias 0 -> 2
- net CANL: track 0.00 -> 40.1 mm, vias 0 -> 1
- net CANH: track 0.00 -> 40.1 mm, vias 0 -> 1
- net RS485_B: track 38.2 -> 0.00 mm, vias 1 -> 0
- net SPI_MOSI: track 0.00 -> 36.4 mm, vias 0 -> 2
- net SPI_MISO: track 0.00 -> 34.1 mm, vias 0 -> 2
- net RS485_A: track 33.8 -> 0.00 mm, vias 1 -> 0
- net SPI_CLK: track 0.00 -> 33.4 mm, vias 0 -> 2
- net MISO: track 33.1 -> 0.00 mm
- net SPI_CS0: track 0.00 -> 32.3 mm, vias 0 -> 2
- net MOSI: track 31.8 -> 0.00 mm
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