File: guhPLC_V0.2.sch (EAGLE design)
At the start: 176 parts, among them IC1 7812DT, IC2 DS2482S-100SOI, K1 62104021021, K2 62104021021, K4 62101021021, K5 61900611021, Q1 BSS123, Q10 BSS123, Q11 BSS123, Q12 FDN360P, Q3 32.768k, Q4 BSS123, Q5 BSS123, Q6 BSS123, Q7 BSS123, Q8 BSS123, Q9 BSS123, U1 LM2672M-3.3, U3 TLC272CD, U4 TLC272CD, U5 ENC28J60/SS, U6 SN65HVD75D, X1 J1006F01P, X2 MKDSN1,5/10-5,08, X3 MKDSN1,5/10-5,08, X4 MKDSN1,5/10-5,08, X5 MKDSN1,5/10-5,08, X6 MKDSN1,5/10-5,08

Commit message: Changed RS485 to CAN Bus - for better multi master communication
Parts:
- removed Q11: BSS123, transistor-small-signal:BSS123
- removed R68, R69: 10, resistor:R-EU_R0603
- removed R70, R71, R72: 10k, resistor:R-EU_R0603
- removed U6: SN65HVD75D, guh:SN65HVD75D
- added C34: 100n, resistor:C-EUC0603
- added C35, C36: 9pF, resistor:C-EUC0603
- added C37, C38: 10u, resistor:C-EUC1206
- added Q2: E3SB16.0000F09G11AE, guh:E3SB16.0000F09G11AE
- added R34, R36, R38: 10k, resistor:R-EU_R0603
- added R37: 18k, resistor:R-EU_R0603
- added U$3: MCP2515-I/SO, guh:MCP2515-I/SO
- added U$4: MCP2551-I/SN, guh:MCP2551-I/SN
- added U2: LD6815TD/18P, guh:LD6815TD/18P
- C6: device resistor:C-EUC0504 -> resistor:C-EUC0603
Connections:
- removed net CS: K4.1, U5.!CS
- removed net DIR: Q11.D, R72.2, U6.!RE, U6.DE
- removed net MISO: K4.4, U5.SO
- removed net MOSI: K4.3, U5.SI
- removed net N$63: R68.1, U6.B
- removed net N$64: R69.1, U6.A
- removed net N$65: Q11.G, R70.1
- removed net RS485_A: R69.2, X2-8.KL
- removed net RS485_B: R68.2, X2-9.KL
- removed net RX: K1.35, R71.1, U6.R
- removed net SCK: K4.2, U5.SCK
- removed net TX: K1.34, R70.2, U6.D
- new net +5V: C38.1, C6.1, U$4.VDD, U2.OUT
- new net CANH: U$4.CANH, X2-7.KL
- new net CANL: U$4.CANL, X2-6.KL
- new net CAN_INT: U$3.~INT
- new net CAN_NRST: R34.2, U$3.~RESET
- new net CAN_OSC1: C35.1, Q2.1, U$3.OSC1
- new net CAN_OSC2: C36.1, Q2.3, U$3.OSC2
- new net CAN_RX: R36.2, U$4.RXD
- new net N$20: U$3.TXCAN, U$4.TXD
- new net N$22: R36.1, R37.1, U$3.RXCAN
- new net N$24: R38.2, U$4.RS
- new net SOM_NRST: K1.2, U$2.PB15/WKUP7/RTC_REFIN/SPI2_MOSI
- new net SPI2_CLK: K4.2, U$3.SCK
- new net SPI2_CS0: K4.1, U$3.~CS
- new net SPI2_MISO: K4.4, U$3.SO
- new net SPI2_MOSI: K4.3, U$3.SI
- new net SPI_CLK: K1.13, U5.SCK
- new net SPI_CS0: K1.14, U5.!CS
- new net SPI_MISO: K1.12, U5.SO
- new net SPI_MOSI: K1.11, U5.SI
- net +3V3: now also C34.1, R34.1, U$3.VDD; no longer C6.1, R71.2, R72.1, U6.VCC
- net 1-WIRE: now also X2-9.KL; no longer X2-6.KL
- net GND: now also C34.2, C35.2, C36.2, C37.2, C38.2, Q2.2, Q2.4, R37.2, R38.1, U$3.VSS, U$4.VSS, U2.GND, X2-8.KL; no longer Q11.S, U6.GND, X2-7.KL
- net VCC: now also C37.1, U2.EN, U2.IN
Other:
- note added: "CAN"
- note removed: "RS485"
- moved on the sheet: C6
